File: main.sch (EAGLE design)
At the start: 116 parts, among them IC1 PM8834-SO08N, IC17 LD398533RM, IC18 LD1117S50TR, IC2 PM8834-SO08N, IC4 CP2102, J1 RJ11, Q1 IRF3205SPBF, Q11 BSS138, Q12 BSS138, Q13 BSS138, Q2 IRF3205SPBF, Q3 IRF3205SPBF, Q4 IRF3205SPBF, Q5 BSS138, Q6 BSS138, Q7 BSS138, Q8 BSS138, Q9 BSS138, T1 SS8050-G, T2 SS8050-G, U1 TMP275AIDR, U4 ESP-WROOM-32, X2 1751248, X4 1751277, X5 1751280

Commit message: Layout
Parts:
- removed C28, C29: 12pF, resistor:C-EUC0805
- removed C56, C62: 100nF, resistor:C-EUC0805
- removed C57: 10nF X7R, resistor:C-EUC0805
- removed C58, C61: 1uF_X5R, resistor:C-EUC0805
- removed C59, C60: 10uF, resistor:CPOL-EUSMCC
- removed D14: BAT60JFILM, diode:DIODE-SOD323-W
- removed IC17: LD398533RM, st-microelectronics:LD398533RM
- removed IC18: LD1117S50TR, v-reg:LD117AS50TR
- removed JP6: (no value), adafruit:PINHD-1X3
- removed LED14: ROOD, led:LEDCHIP-LED0805
- removed LED2: RGBLED5050, adafruit:RGBLED5050
- removed R44, R45: 10K, resistor:R-EU_R0805
- removed R46: 10R, resistor:R-EU_R0805
- removed R47: X, resistor:R-EU_R0805
- removed R48: 1K, resistor:R-EU_R0805
- removed U4: ESP-WROOM-32, esp32:ESP-WROOM-32
- removed X4: 1751277, con-phoenix-350:1751277
- removed X5: 1751280, con-phoenix-350:1751280
- added C17, C18, C20: 100n, resistor:C-EUC0805
- added C19, C7: 100nF, resistor:C-EUC0805
- added C21, C22: 1uF X7R, resistor:C-EUC0805
- added C9: (no value), resistor:CPOL-EUSMCA
- added IC3: CP2102, silabs:CP2102
- added IC5: PM8834-SO08N, PM8834:PM8834-SO08N
- added JP2: (no value), adafruit:PINHD-1X3
- added LED1: RGBLED5050, adafruit:RGBLED5050
- added U2: TMP275AIDR, TMP275AIDR:TMP275AIDR
- added X1: 1751248, con-phoenix-350:1751248
- added X3: 1751277, con-phoenix-350:1751277
- C1: value 100n -> 10uF; device resistor:C-EUC0805 -> resistor:CPOL-EUSMCC
- C10: value 100n -> 1uF_X5R
- C11: value (none) -> 100nF; device resistor:CPOL-EUSMCA -> resistor:C-EUC0805
- C14, C15: value 100n -> 12pF
- C2: value 100nF -> 10uF; device resistor:C-EUC0805 -> resistor:CPOL-EUSMCC
- C3: value 100nF -> 1uF_X5R
- C5: value 1uF_X5R -> 10nF X7R
- C6: value 1uF X7R -> 1uF_X5R
- C8: value 1uF X7R -> 100nF
- D1, D2: value BAT54S -> BAT60JFILM; device diode:BAT54S -> diode:DIODE-SOD323-W
- D5: value BAT60JFILM -> BAT54S; device diode:DIODE-SOD323-W -> diode:BAT54S
- IC1: value PM8834-SO08N -> LD1117S50TR; device PM8834:PM8834-SO08N -> v-reg:LD117AS50TR
- IC2: value PM8834-SO08N -> LD398533RM; device PM8834:PM8834-SO08N -> st-microelectronics:LD398533RM
- IC4: value CP2102 -> PM8834-SO08N; device silabs:CP2102 -> PM8834:PM8834-SO08N
- Q1: value IRF3205SPBF -> (none); device IRF3205SPBF:IRF3205SPBF -> crystal:CRYSTALTC38H
- Q10: value (none) -> IRF3205SPBF; device crystal:CRYSTALTC38H -> IRF3205SPBF:IRF3205SPBF
- Q11, Q12, Q13: value BSS138 -> IRF3205SPBF; device SparkFun:MOSFET-NCHANNELSMD -> IRF3205SPBF:IRF3205SPBF
- Q2, Q3, Q4: value IRF3205SPBF -> BSS138; device IRF3205SPBF:IRF3205SPBF -> SparkFun:MOSFET-NCHANNELSMD
- R1: value 10K -> 22K1
- R10: value 10R -> 10K
- R11, R12, R29: value 10K -> 4K7
- R15, R16: value X -> 10K
- R17, R18, R38, R39: value 1K -> 10K
- R2: value 10R -> 47K5
- R21, R22: value 10K -> X
- R23, R24: value 10K -> 10R
- R25, R26, R34: value 10K -> 1K
- R3, R4: value 4K7 -> 1K
- R31, R32: value 0R -> 10K
- R33: value 2K -> 10K
- R35: value 22K1 -> 10K
- R36: value 47K5 -> 10K
- R5: value 4K7 -> 2K
- R7, R8: value 1K -> 0R
- S1: value (none) -> MOMENTARY-SWITCH-SPST-SMD-5.2-REDUNDANT; device switch-omron:10-XX -> SparkFun-Switches:MOMENTARY-SWITCH-SPST-SMD-5.2-REDUNDANT
- U1: value TMP275AIDR -> ESP-WROOM-32; device TMP275AIDR:TMP275AIDR -> esp32:ESP-WROOM-32
- X2: value 1751248 -> 1751280; device con-phoenix-350:1751248 -> con-phoenix-350:1751280
- renumbered C30 to C16, CN2 to CN1, S3 to S2
Connections:
- removed net LED: U4.IO27
- removed net N$22: X5-1.K
- removed net N$28: Q13.D, R41.1
- removed net N$30: LED2.RED_C, R40.1
- removed net N$33: D3.C1A2, R46.2, R48.1
- removed net N$37: Q12.G
- removed net N$4: X5-4.K
- removed net N$40: Q11.G
- removed net N$41: Q9.G
- removed net N$99: LED14.A, R39.1
- new net LEDB: Q8.G, U1.IO27
- new net LEDG: Q7.G, U1.IO26
- new net LEDR: Q6.G, U1.IO25
- new net P1: Q9.D, R35.1, U1.IO13
- net +12V: now also C1.+, C21.1, C22.1, IC1.IN, IC4.VCC, IC5.VCC, R38.2, R39.2, R42.2, R43.2, X1-1.K, X3-1.K; no longer C59.+, C6.1, C8.1, IC1.VCC, IC18.IN, IC2.VCC, R11.2, R12.2, R13.2, R14.2, X2-1.K, X4-1.K
- net +3V3: now also C10.1, C11.1, C19.1, C6.1, C7.1, C8.1, C9.+, D4.C2, IC2.VO, IC3.REGIN, IC3.VDD, LED1.BLUE_A, LED1.GREEN_A, LED1.RED_A, Q2.G, Q3.G, Q4.G, R11.2, R12.2, R13.1, R15.1, R17.1, R19.1, R27.2, R28.2, R29.2, R35.2, U1.3V3, U2.V+; no longer C11.+, C12.1, C13.1, C4.1, C5.1, C61.1, C62.1, D1.C2, D2.C2, IC17.VO, IC4.REGIN, IC4.VDD, LED2.BLUE_A, LED2.GREEN_A, LED2.RED_A, Q6.G, Q7.G, Q8.G, R1.2, R23.1, R25.1, R27.1, R29.1, R33.2, R41.2, R6.2, R7.2, R8.2, R9.2, U1.V+, U4.3V3
- net +5V: now also C3.1, C4.1, D1.C, D2.C, D5.C2, IC2.VIN, IC2.VINH, JP1.1, R14.1, R33.2, X2-1.K, X2-4.K; no longer C56.1, C58.1, D14.C, D4.C2, D5.C, IC17.VIN, IC17.VINH, JP6.1, R24.1, R37.2
- net BTN: now also C13.1, R4.1, S1.2, U1.IO34; no longer C2.1, R8.1, S1.S, U4.IO34
- net CTS: now also IC3.CTS; no longer IC4.CTS
- net DCD: now also IC3.DCD; no longer IC4.DCD
- net DSR: now also IC3.DSR; no longer IC4.DSR
- net DTR: now also IC3.DTR, R9.1; no longer IC4.DTR, R42.1
- net EN: now also C12.1, R3.1, U1.EN; no longer C3.1, R7.1, U4.EN
- net GND: now also C1.-, C11.2, C17.2, C18.2, C19.2, C2.-, C20.2, C21.2, C22.2, C7.2, C9.-, D5.A1, IC1.ADJ, IC3.GND, IC3.GND@EXP, IC3.GND@M, IC5.GND, JP2.3, Q10.S, Q6.S, Q7.S, Q8.S, R2.1, R21.1, R22.1, R36.2, R37.2, R40.2, R41.2, R6.2, S1.1, U1.GND@1, U1.GND@15, U1.GND@38, U2.A0, U2.A1, U2.A2, U2.GND, X1-2.K, X2-3.K, X2-6.K; no longer C1.2, C11.-, C2.2, C28.2, C29.2, C56.2, C57.2, C58.2, C59.-, C60.-, C61.2, C62.2, D1.A1, D2.A1, IC1.GND, IC17.GND, IC18.ADJ, IC4.GND@EXP, IC4.GND@M, JP6.3, LED14.C, Q1.S, Q2.S, Q3.S, Q4.S, R15.1, R16.1, R19.2, R20.2, R21.2, R22.2, R34.2, R36.1, R47.1, S1.P, U1.A0, U1.A1, U1.A2, U1.GND, U4.GND@1, U4.GND@15, U4.GND@38, X2-2.K, X5-3.K, X5-6.K
- net HV: now also JP2.1, R16.1, R18.1, R20.1; no longer JP1.1, R26.1, R28.1, R30.1
- net HV1: now also JP1.2, Q2.D, R14.2; no longer JP6.2, Q5.D, R24.2
- net HV2: now also JP2.2, Q3.D, R16.2; no longer JP1.2, Q6.D, R26.2
- net HV3: now also Q4.D, R18.2; no longer Q7.D, R28.2
- net HV4: now also Q5.D, R20.2; no longer Q8.D, R30.2
- net I2C_SCL: now also R12.1, U1.IO22, U2.SCL; no longer R4.1, U1.SCL, U4.IO22
- net I2C_SDA: now also R11.1, U1.IO23, U2.SDA; no longer R3.1, U1.SDA, U4.IO23
- net INP1: now also C17.1, R25.2, R27.1, U1.IO14; no longer C10.1, R17.2, R9.1, U4.IO26
- net INP2: now also C18.1, R26.2, R28.1, U1.IO12; no longer C1.1, C15.1, R1.1, R18.2, R48.2, R6.1, U4.IO25
- net IO0: now also U1.IO0; no longer U4.IO0
- net LV0: now also Q2.S, R13.2; no longer Q5.S, R23.2
- net LV1: now also Q3.S, R15.2; no longer Q6.S, R25.2
- net LV2: now also Q4.S, R17.2; no longer Q7.S, R27.2
- net LV3: now also Q5.S, R19.2; no longer Q8.S, R29.2
- net N$1: now also Q6.D, R30.2; no longer Q9.D, R40.2
- net N$10: now also IC4.IN2, R38.1; no longer IC1.IN2, R11.1
- net N$102: now also C5.1, IC2.BYPASS; no longer C57.1, IC17.BYPASS
- net N$11: now also LED1.RED_C, R31.1; no longer LED2.GREEN_C, R44.1
- net N$12: now also IC4.OUT1, Q11.G; no longer IC1.OUT1, Q2.G
- net N$13: now also IC4.OUT2, Q10.G; no longer IC1.OUT2, Q1.G
- net N$14: now also Q11.D, X3-3.K; no longer Q2.D, X4-3.K
- net N$15: now also IC5.OUT1, Q13.G; no longer IC2.OUT1, Q4.G
- net N$16: now also IC5.OUT2, Q12.G; no longer IC2.OUT2, Q3.G
- net N$17: now also Q12.D, X3-4.K; no longer Q3.D, X4-4.K
- net N$18: now also Q13.D, X3-5.K; no longer Q4.D, X4-5.K
- net N$19: now also IC3.!SUSPEND, R6.1; no longer IC4.!SUSPEND, R34.1
- net N$2: now also R22.2, R24.1, X2-5.K; no longer R15.2, R2.1, X5-5.K
- net N$20: now also R21.2, R23.1, X2-2.K; no longer R10.1, R16.2, X5-2.K
- net N$2001: now also IC5.IN2, R43.1; no longer IC2.IN2, R14.1
- net N$21: now also IC3.!RST, R5.1; no longer IC4.!RST, R33.1
- net N$23: now also C2.+, D1.A, IC1.OUT; no longer C60.+, D14.A, IC18.OUT, R39.2
- net N$24: now also IC3.VBUS, R1.2, R2.2; no longer IC4.VBUS, R35.2, R36.2
- net N$25: now also IC3.D-; no longer IC4.D-
- net N$26: now also R33.1, R34.1; no longer R37.1, R38.1
- net N$27: now also C20.1, D5.C1A2, Q9.G, R34.2; no longer C14.1, D4.C1A2, Q13.G, R38.2
- net N$29: now also LED1.BLUE_C, R32.1; no longer LED2.BLUE_C, R45.1
- net N$2OO: now also IC5.EN1, R42.1; no longer IC2.EN1, R13.1
- net N$3: now also D3.C1A2, R23.2, R25.1; no longer D2.C1A2, R10.2, R17.1
- net N$31: now also Q7.D, R31.2; no longer Q11.D, R44.2
- net N$32: now also Q8.D, R32.2; no longer Q12.D, R45.2
- net N$38: now also C14.1, Q1.2, U1.IO32; no longer C28.1, Q10.2, U4.IO32
- net N$39: now also C15.1, Q1.1, U1.IO33; no longer C29.1, Q10.1, U4.IO33
- net N$42: now also R9.2; no longer R42.2
- net N$43: now also R10.2; no longer R43.2
- net N$5: now also LED1.GREEN_C, R30.1; no longer R46.1, R47.2
- net N$6: now also IC3.D+; no longer IC4.D+
- net N$7: now also Q10.D, X3-2.K; no longer Q1.D, X4-2.K
- net N$8: now also D4.C1A2, R24.2, R26.1; no longer D1.C1A2, R18.1, R2.2
- net N$9: now also IC4.EN1, R39.1; no longer IC1.EN1, R12.1
- net PWM0: now also IC4.IN1, R36.1, U1.IO17; no longer IC1.IN1, R22.1, U4.IO17
- net PWM1: now also IC4.EN2, R37.1, U1.IO5; no longer IC1.EN2, R21.1, U4.IO5
- net PWM2: now also IC5.IN1, R40.1, U1.IO18; no longer IC2.IN1, R20.1, U4.IO18
- net PWM3: now also IC5.EN2, R41.1, U1.IO19; no longer IC2.EN2, R19.1, U4.IO19
- net RI: now also IC3.RI; no longer IC4.RI
- net RTS: now also IC3.RTS, R10.1; no longer IC4.RTS, R43.1
- net RXD: now also IC3.RXD, R8.1; no longer IC4.RXD, R32.1
- net RXD0: now also R7.2, U1.RXD0; no longer R31.2, U4.RXD0
- net TEMP_ALERT: now also R29.1, U1.IO21, U2.ALERT; no longer R5.1, U1.ALERT, U4.IO21
- net TXD: now also IC3.TXD, R7.1; no longer IC4.TXD, R31.1
- net TXD0: now also R8.2, U1.TXD0; no longer R32.2, U4.TXD0
- net VBUS: now also D2.A, R1.1; no longer D5.A, R35.1
