File: prog.brd (EAGLE design)
At the start: 160 x 100 mm, 49 parts, among them IC2 LD398533RM, IC3 74AHCT1G04DBV, Q1 220mA/50V/3.5Ω, T1 SS8050-G, T2 SS8050-G, U1 SN74AHC125PWR, U2 FT2232HL-REEL

Commit message: work on programmer board
Parts:
- removed R7, R8, R9: 33R, resistor:R0805
- added C15, C16: 12pF, resistor:C0805
- added C17, C18, C20, C22: 4u7, resistor:C0805
- added C19, C21, C23, C24, C25, C26, C27, C28, C29: 100n, resistor:C0805
- added L1, L2: BLM15HB221SN1, inductors:0402
- added LED2: GREEN, led:CHIPLED_0805
- added LED3: BLUE, led:CHIPLED_0805
- added Q2: (no value), crystal:HC49UP
- added R19, R20: 2K2, resistor:R0805
- added R21: 12K, resistor:R0805
- added R22: 1K, resistor:R0805
- moved C14 314.0 mm to (131.4, 10.2), turned to 180 degrees
- moved C13 282.5 mm to (134.6, -17.5), turned to 270 degrees
- moved D3 281.1 mm to (140.0, -17.5)
- moved R16 274.2 mm to (136.8, -17.5), turned to 90 degrees
- moved C11 248.1 mm to (134.0, -26.0)
- moved D1 248.1 mm to (139.7, -26.0)
- moved Q1 248.1 mm to (130.8, -26.0)
- moved R15 248.1 mm to (136.5, -26.0)
- moved U1 238.1 mm to (131.4, 6.03)
- moved R18 228.5 mm to (131.4, -140.0)
- moved R17 225.8 mm to (127.0, -130.8)
- moved J2 190.2 mm to (146.4, 6.67), turned to 90 degrees
- moved J1 189.0 mm to (148.9, 16.5), turned to 90 degrees
- moved R5 158.2 mm to (121.3, 45.4)
- moved R6 157.6 mm to (116.2, 45.1)
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Connections:
- removed net AGND: U2.10
- removed net N$3: R7.2, U2.63
- removed net N$5: R9.2, U2.61
- removed net N$6: R8.2, U2.62
- removed net VCCIO-1: U2.20
- removed net VCCIO-2: U2.31
- removed net VCCIO-3: U2.42
- removed net VCCIO-4: U2.56
- removed net VCORE-1: U2.12
- removed net VCORE-2: U2.37
- removed net VCORE-3: U2.64
- removed net VPHY: U2.4
- removed net VPLL: U2.9
- removed net VREGIN: U2.50
- removed net VREGOUT: U2.49
- new net +1V8: C18.1, C27.1, C28.1, C29.1, U2.12, U2.37, U2.49, U2.64
- new net N$11: LED3.A, R20.1
- new net N$12: LED2.A, R19.1
- new net N$13: C15.1, Q2.1, U2.2
- new net N$14: C16.1, Q2.2, U2.3
- new net N$15: R22.2, U2.14
- new net N$16: R21.2, U2.6
- new net N$17: U2.8
- new net N$18: U2.7
- new net N$19: C19.1, C20.1, L2.2, U2.9
- new net N$20: C21.1, C22.1, L1.2, U2.4
- net !FT_RXLED: now also LED3.C
- net !FT_TXLED: now also LED2.C
- net +3V3: now also C17.1, C23.1, C24.1, C25.1, C26.1, L1.1, L2.1, R19.2, R20.2, R22.1, U2.20, U2.31, U2.42, U2.50, U2.56
- net EECLK: now also U2.62; no longer R8.1
- net EECS: now also U2.63; no longer R7.1
- net EEDATA: now also U2.61; no longer R9.1
- net FT_TCK: now also U2.16
- net FT_TDI: now also U2.17
- net FT_TDO: now also U2.18
- net FT_TMS: now also U2.19
- net GND: now also C15.2, C16.2, C17.2, C18.2, C19.2, C20.2, C21.2, C22.2, C23.2, C24.2, C25.2, C26.2, C27.2, C28.2, C29.2, R21.1, U2.10, U2.13
Routing:
- net EECS: track 0.00 -> 12.4 mm
- net EECLK: track 0.00 -> 8.88 mm
- net N$4: track 0.00 -> 6.63 mm
- net +3V3: track 0.00 -> 4.45 mm
- net EEDATA: track 0.00 -> 3.35 mm
- added copper zone on layer 1, net GND
