File: rgb-controller.brd (EAGLE design)
At the start: 100 x 50 mm, 85 parts, among them IC1 LD1117S50TR, IC2 LD398533RM, IC4 PM8834-SO08N, IC5 PM8834-SO08N, J1 RJ11, Q10 IRF3205SPBF, Q11 IRF3205SPBF, Q12 IRF3205SPBF, Q13 IRF3205SPBF, Q2 BSS138, Q3 BSS138, Q6 BSS138, Q9 BSS138, U1 ESP-WROOM-32, U2 TMP275AIDR, U3 TSL2561T, X1 1751248, X2 1751280, X3 1751277

Commit message: eagle
Parts:
- removed C14, C15: 12pF, resistor:C0805
- removed C19, C4, C7: 100nF, resistor:C0805
- removed C20: 100n, resistor:C0805
- removed C3, C6: 1uF_X5R, resistor:C0805
- removed C5: 10nF X7R, resistor:C0805
- removed IC2: LD398533RM, st-microelectronics:SOT23-5L
- removed J1: RJ11, SparkFun-Connectors:RJ11-6
- removed Q1: (no value), crystal:TC38H
- removed Q6, Q9: BSS138, SparkFun:SOT23-3
- removed R33, R35: 10K, resistor:R0805
- removed R34: 1K, resistor:R0805
- removed S2: MOMENTARY-SWITCH-SPST-SMD-5.2-REDUNDANT, SparkFun-Switches:TACTILE_SWITCH_SMD_5.2MM
- removed U2: TMP275AIDR, TMP275AIDR:SOIC127P600X175-8N
- added C11, C24: 10uF, resistor:SMC_C
- added C47: 100nF, resistor:C0805
- added C49: 10uF, resistor:C0805
- added C9: 15nF, resistor:C0805
- added D2: MMSZ5240BT1G, diode:SOD123
- added D6: SMAJ12A, diode:DO-214AC
- added Q4: IRFR5305, transistor-power:D-PAK_TO252AA
- added R2, R5: 10K, resistor:R0805
- added S3: B3S-10XX, clock:B3S-10XX
- added U14: PCT2075D, clock:SOIC8_150MIL
- added U4: LD117AS33TR, v-reg:SOT223
- D5: value BAT54S -> BAT60JFILM; device diode:SOT23 -> diode:SOD323-W
- H1, H2, H3, H4: value MOUNT-HOLE3.0 -> MOUNT-HOLE3.2; device holes:3,0 -> holes:3,2
- S1: value MOMENTARY-SWITCH-SPST-SMD-5.2-REDUNDANT -> B3S-10XX; device SparkFun-Switches:TACTILE_SWITCH_SMD_5.2MM -> clock:B3S-10XX
- moved S1 74.4 mm to (18.7, -41.3), turned to 0 degrees
- moved J3 55.4 mm to (-50.8, -44.8)
- moved J2 47.8 mm to (-32.4, -46.4)
- moved D5 29.7 mm to (-0.95, -16.2), turned to 90 degrees
- moved C1 10.5 mm to (4.76, -11.1)
- moved C2 10.5 mm to (4.76, -21.9)
- moved IC1 10.5 mm to (4.76, -16.5)
- moved D1 10.2 mm to (-0.95, -21.3)
- moved C16 1.14 mm to (9.84, -5.08)
- moved R1 1.14 mm to (9.84, -7.30)
Connections:
- removed net N$1: Q6.3, R30.2
- removed net N$102: C5.1, IC2.4
- removed net N$26: J1.5, R33.1, R34.1
- removed net N$27: C20.1, D5.3, Q9.1, R34.2
- removed net N$38: C14.1, Q1.2, U1.8
- removed net N$39: C15.1, Q1.1, U1.9
- removed net P1: Q9.3, R35.1, U1.26
- new net N$113: C11.+, D1.C, D5.C, U4.3
- new net N$40: C9.1, D2.A, Q4.1, R2.2
- new net VIN: D6.C, Q4.4, X1.1
- net +12V: now also D2.C, Q4.3; no longer X1.1
- net +3V3: now also C24.+, C47.1, C49.1, R5.2, U14.8, U4.4; no longer C19.1, C6.1, C7.1, IC2.5, LED1.A, R35.2, U2.8
- net +5V: no longer C3.1, C4.1, D1.C, D5.2, IC2.1, IC2.3, J1.2, R33.2
- net BTN: now also S1.1; no longer S1.3, S1.4
- net ESP_IO0: now also R5.1, S3.1; no longer S2.3, S2.4
- net GND: now also C11.-, C24.-, C47.2, C49.2, C9.2, D6.A, R2.1, R30.2, S1.3, S1.4, S3.3, S3.4, U14.4, U14.5, U14.6, U14.7, U4.1; no longer C14.2, C15.2, C19.2, C20.2, C3.2, C4.2, C5.2, C6.2, C7.2, D5.1, IC2.2, J1.3, Q6.2, Q9.2, S1.1, S1.2, S2.1, S2.2, U2.4, U2.5, U2.6, U2.7
- net I2C_SCL: now also U14.2; no longer U2.2
- net I2C_SDA: now also U14.1; no longer U2.1
- net LEDR: now also LED1.A; no longer Q6.1
Routing:
- net VIN: track 0.00 -> 36.0 mm, vias 0 -> 1
- net +5V: track 84.4 -> 49.0 mm
- net P1: track 35.4 -> 0.00 mm, vias 2 -> 0
- net ESP_RXD0: track 37.3 -> 3.64 mm
- net N$23: track 31.9 -> 0.78 mm, vias 2 -> 0
- net ESP_TXD0: track 34.7 -> 3.58 mm
- net ESP_EN: track 53.0 -> 23.6 mm
- net +3V3: track 182.6 -> 158.9 mm, vias 12 -> 11
- net LV0: track 55.0 -> 31.5 mm, vias 4 -> 3
- net ESP_TDI: track 30.0 -> 10.1 mm
- net ESP_TDO: track 18.7 -> 2.18 mm
- net ESP_TCK: track 22.8 -> 8.98 mm
- net N$4: track 13.2 -> 0.00 mm, vias 1 -> 0
- net N$38: track 12.8 -> 0.00 mm
- net ESP_TMS: track 24.0 -> 11.7 mm
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- removed copper zone on layer 16, net +12V
Other:
- outline, holes or cut-outs redrawn
