File: rgb-controller.sch (EAGLE design)
At the start: 85 parts, among them IC1 LD1117S50TR, IC2 LD398533RM, IC4 PM8834-SO08N, IC5 PM8834-SO08N, J1 RJ11, Q10 IRF3205SPBF, Q11 IRF3205SPBF, Q12 IRF3205SPBF, Q13 IRF3205SPBF, Q2 BSS138, Q3 BSS138, Q6 BSS138, Q9 BSS138, U1 ESP-WROOM-32, U2 TMP275AIDR, U3 TSL2561T, X1 1751248, X2 1751280, X3 1751277

Commit message: eagle
Parts:
- removed C14, C15: 12pF, resistor:C-EUC0805
- removed C19, C4, C7: 100nF, resistor:C-EUC0805
- removed C20: 100n, resistor:C-EUC0805
- removed C3, C6: 1uF_X5R, resistor:C-EUC0805
- removed C5: 10nF X7R, resistor:C-EUC0805
- removed IC2: LD398533RM, st-microelectronics:LD398533RM
- removed J1: RJ11, SparkFun-Connectors:RJ11-6
- removed Q1: (no value), crystal:CRYSTALTC38H
- removed Q6, Q9: BSS138, SparkFun:MOSFET-NCHANNELSMD
- removed R33, R35: 10K, resistor:R-EU_R0805
- removed R34: 1K, resistor:R-EU_R0805
- removed S2: MOMENTARY-SWITCH-SPST-SMD-5.2-REDUNDANT, SparkFun-Switches:MOMENTARY-SWITCH-SPST-SMD-5.2-REDUNDANT
- removed U2: TMP275AIDR, TMP275AIDR:TMP275AIDR
- added C11, C24: 10uF, resistor:CPOL-EUSMCC
- added C47: 100nF, resistor:C-EUC0805
- added C49: 10uF, resistor:C-EUC0805
- added C9: 15nF, resistor:C-EUC0805
- added D2: MMSZ5240BT1G, diode:DIODE-SOD123
- added D6: SMAJ12A, diode:DIODE-DO-214AC
- added Q4: IRFR5305, transistor-power:IRFR5305
- added R2, R5: 10K, resistor:R-EU_R0805
- added S3: B3S-10XX, clock:B3S-10XX
- added U14: PCT2075D, clock:PCT2075D
- added U4: LD117AS33TR, v-reg:LD117AS33TR
- D5: value BAT54S -> BAT60JFILM; device diode:BAT54S -> diode:DIODE-SOD323-W
- H1, H2, H3, H4: value MOUNT-HOLE3.0 -> MOUNT-HOLE3.2; device holes:MOUNT-HOLE3.0 -> holes:MOUNT-HOLE3.2
- S1: value MOMENTARY-SWITCH-SPST-SMD-5.2-REDUNDANT -> B3S-10XX; device SparkFun-Switches:MOMENTARY-SWITCH-SPST-SMD-5.2-REDUNDANT -> clock:B3S-10XX
Connections:
- removed net N$1: Q6.D, R30.2
- removed net N$102: C5.1, IC2.BYPASS
- removed net N$26: J1.5, R33.1, R34.1
- removed net N$27: C20.1, D5.C1A2, Q9.G, R34.2
- removed net N$38: C14.1, Q1.2, U1.IO32
- removed net N$39: C15.1, Q1.1, U1.IO33
- removed net P1: Q9.D, R35.1, U1.IO4
- new net N$113: C11.+, D1.C, D5.C, U4.IN
- new net N$40: C9.1, D2.A, Q4.G, R2.2
- new net VIN: D6.C, Q4.D, X1-1.K
- net +12V: now also D2.C, Q4.S; no longer X1-1.K
- net +3V3: now also C24.+, C47.1, C49.1, R5.2, U14.VCC, U4.OUT; no longer C19.1, C6.1, C7.1, IC2.VO, LED1.A, R35.2, U2.V+
- net +5V: no longer C3.1, C4.1, D1.C, D5.C2, IC2.VIN, IC2.VINH, J1.2, R33.2
- net BTN: now also S1.P; no longer S1.2
- net ESP_IO0: now also R5.1, S3.P; no longer S2.2
- net GND: now also C11.-, C24.-, C47.2, C49.2, C9.2, D6.A, R2.1, R30.2, S1.S, S1.S1, S3.S, S3.S1, U14.A0, U14.A1, U14.A2, U14.GND, U4.ADJ; no longer C14.2, C15.2, C19.2, C20.2, C3.2, C4.2, C5.2, C6.2, C7.2, D5.A1, IC2.GND, J1.3, Q6.S, Q9.S, S1.1, S2.1, U2.A0, U2.A1, U2.A2, U2.GND
- net I2C_SCL: now also U14.SCL; no longer U2.SCL
- net I2C_SDA: now also U14.SDA; no longer U2.SDA
- net LEDR: now also LED1.A; no longer Q6.G
Other:
- note added: "7-bit I2C Address is 0x48"
